File: hardware/kicad/canarynode.kicad_sch (KiCad schematic)
At the start: 0 parts

Commit message: schematic: TPS62160 buck subcircuit complete (5V to 3.3V/1A)
TPS62160DGKR adjustable buck, VSSOP-8 (C60726)
- L=3.3uH XFL3012-332MEC for low-VIN operation per datasheet 9.2.2.4
- C1=10uF/10V X5R 0603 (C19702), C2=22uF/6.3V X5R 0603 (C59461)
- FB divider: R1=562k, R2=180k for Vout=3.30V per Eq 6 (Vref=0.8V)
- R3=100k PG pull-up to +3.3V; PG net labeled for future GPIO/test point
- VOS routed to VOUT at output cap per 11.1 layout guidance
- PGND/AGND single-point ground at IC
- PWR_FLAGs on +5V, +3.3V, GND
- Footprints: KiCad built-ins + Coilcraft_Local for XFL3012
- ERC: 0 errors
Parts:
- added C1: 10u, Capacitor_SMD:C_0603_1608Metric, symbol Device:C
- added C2: 22u, Capacitor_SMD:C_0603_1608Metric, symbol Device:C
- added L1: 3.3u, Coilcraft_Local:IND_XFL3012_COC, symbol Device:L
- added R1: 562k, Resistor_SMD:R_0402_1005Metric, symbol Device:R
- added R2: 180k, Resistor_SMD:R_0402_1005Metric, symbol Device:R
- added R3: 100k, Resistor_SMD:R_0402_1005Metric, symbol Device:R
- added U1: TPS62160DGK, Package_SO:MSOP-8_3x3mm_P0.65mm, symbol Regulator_Switching:TPS62160DGK
Connections:
- new net: R1.2, R2.1, U1.5 (FB)
- new net: L1.1, U1.7 (SW)
- new net +3.3V: C2.1, L1.2, R1.1, R3.1, U1.6 (VOS)
- new net +5V: C1.1, U1.2 (VIN), U1.3 (EN)
- new net GND: C1.2, C2.2, R2.2, U1.1 (PGND), U1.4 (AGND)
- new net PG: R3.2, U1.8 (PG)
Other:
- note added: "EN tied to VIN: buck always-on when VBUS present"
